Commit message: modifications

File: ldlidar_node/urdf/ldlidar_descr.urdf.xacro (robot description, xacro)
@@ -16,5 +16,5 @@
             <origin xyz="0 0 0" rpy="0 0 0"/>
             <geometry>
-                <mesh filename="package://ldlidar_node/urdf/model/LD19.stl" scale="0.001 0.001 0.001" />
+                <mesh filename="file://$(find ldrobot-lidar-ros2_nw_arch)/3d_model/LD19.stl" scale="0.001 0.001 0.001" />
             </geometry>
             <material name="ldlidar_mat">
